File: Hardware/Rev2_1/MPPT_String.sch (KiCad schematic (older format))
At the start: 5 parts, among them Q4 2N7002K, U1 LTC4411

Commit message: Adding initial MPPT design files and updated documentation. May need some more work to clean up but mostly there.
Changed lines of the file:
@@
 $Descr A 11000 8500
 encoding utf-8
-Sheet 27 37
+Sheet 2 37
 Title "Fox-1 Maximum Power Point Tracker"
-Date "30 nov 2015"
+Date "3 sep 2016"
 Rev "2.0"
 Comp "The Radio Amateur Satellite Corporation"
@@
 AR Path="/534CE2A8/5347F386" Ref="#PWR0197"  Part="1"
 AR Path="/549391D0/5347F386" Ref="#PWR0181"  Part="1"
-F 0 "#PWR0235" H 1850 2150 30  0001 C CNN
+F 0 "#PWR029" H 1850 2150 30  0001 C CNN
 F 1 "GND" H 1850 2080 30  0001 C CNN
 F 2 "" H 1850 2150 60  0000 C CNN
@@
 AR Path="/534CE2A8/534E3EEE" Ref="U20"  Part="1"
 AR Path="/549391D0/534E3EEE" Ref="U17"  Part="1"
-F 0 "U11" H 7250 2375 50  0000 C CNN
+F 0 "U1" H 7250 2375 50  0000 C CNN
 F 1 "LTC4411" H 7350 2300 50  0000 C CNN
 F 2 "TSOT23-5" H 7400 2225 50  0000 C CNN
@@
 AR Path="/534CE2A8/534E3EF8" Ref="#PWR0198"  Part="1"
 AR Path="/549391D0/534E3EF8" Ref="#PWR0182"  Part="1"
-F 0 "#PWR0236" H 6900 2000 30  0001 C CNN
+F 0 "#PWR030" H 6900 2000 30  0001 C CNN
 F 1 "GND" H 6900 1930 30  0001 C CNN
 F 2 "" H 6900 2000 60  0000 C CNN
@@
 AR Path="/534CE2A8/534E3F02" Ref="#PWR0199"  Part="1"
 AR Path="/549391D0/534E3F02" Ref="#PWR0183"  Part="1"
-F 0 "#PWR0237" H 8000 2400 30  0001 C CNN
+F 0 "#PWR031" H 8000 2400 30  0001 C CNN
 F 1 "GND" H 8000 2330 30  0001 C CNN
 F 2 "" H 8000 2400 60  0000 C CNN
@@
 AR Path="/534CE2A8/534FC4F2" Ref="#FLG0200"  Part="1"
 AR Path="/549391D0/534FC4F2" Ref="#FLG0184"  Part="1"
-F 0 "#FLG0238" H 2500 1795 30  0001 C CNN
+F 0 "#FLG032" H 2500 1795 30  0001 C CNN
 F 1 "PWR_FLAG" H 2500 1880 30  0000 C CNN
 F 2 "" H 2500 1700 60  0000 C CNN
@@
 AR Path="/534CE2A8/53895782" Ref="R200"  Part="1"
 AR Path="/549391D0/53895782" Ref="R198"  Part="1"
-F 0 "R194" H 5850 5200 50  0000 C CNN
+F 0 "R190" H 5850 5200 50  0000 C CNN
 F 1 "10K" H 5825 5125 50  0000 C CNN
 F 2 "R0402" H 5875 5050 50  0000 C CNN
@@
 AR Path="/534CE2A8/53895792" Ref="#PWR0201"  Part="1"
 AR Path="/549391D0/53895792" Ref="#PWR0185"  Part="1"
-F 0 "#PWR0239" H 6350 5950 30  0001 C CNN
+F 0 "#PWR033" H 6350 5950 30  0001 C CNN
 F 1 "GND" H 6350 5880 30  0001 C CNN
 F 2 "" H 6350 5950 60  0000 C CNN
@@
 AR Path="/534CE2A8/53895C9A" Ref="R199"  Part="1"
 AR Path="/549391D0/53895C9A" Ref="R197"  Part="1"
-F 0 "R193" H 6500 4475 50  0000 C CNN
+F 0 "R189" H 6500 4475 50  0000 C CNN
 F 1 "10K" H 6475 4400 50  0000 C CNN
 F 2 "R0402" H 6525 4325 50  0000 C CNN
@@
 AR Path="/534CE2A8/54818CE4" Ref="Q18"  Part="1"
 AR Path="/549391D0/54818CE4" Ref="Q17"  Part="1"
-F 0 "Q12" H 6475 5625 50  0000 R CNN
+F 0 "Q4" H 6475 5625 50  0000 R CNN
 F 1 "2N7002K" H 6725 5550 50  0000 R CNN
 F 2 "SOT23" H 6500 5475 50  0000 C CNN
@@
 AR Path="/534CD3EE/565CA5CA" Ref="D10"  Part="1"
 AR Path="/534CE2A1/565CA5CA" Ref="D12"  Part="1"
-F 0 "D9" V 5650 4500 50  0000 C CNN
+F 0 "D7" V 5650 4500 50  0000 C CNN
 F 1 "SDM10U45-7" V 5725 4300 50  0000 C CNN
 F 2 "SOD523" V 5800 4400 50  0000 C CNN
