File: Hardware/Rev2_1/RTD_Measurement.sch (KiCad schematic (older format))
At the start: 36 parts, among them U3 LM6144A

Commit message: Adding initial MPPT design files and updated documentation. May need some more work to clean up but mostly there.
Other:
- note removed: "Capacitor not on PCB,\nstack ontop of feedback resistor"
